File: resources/kicad/xiao_lamp.kicad_sch (KiCad schematic)
At the start: 14 parts, among them U1 LM78M05_TO252, U2 SeeeduinoXIAO

Commit message: поправлена схема
Parts:
- removed R2: 100K, Resistor_SMD:R_1206_3216Metric, symbol Device:R
Changed lines of the file:
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@@
   (junction (at 71.12 46.99) (diameter 0) (color 0 0 0 0)
   )
-  (junction (at 252.73 82.55) (diameter 0) (color 0 0 0 0)
-  )
   (junction (at 38.1 46.99) (diameter 0) (color 0 0 0 0)
   )
@@
     (stroke (width 0) (type default))
   )
-  (wire (pts (xy 252.73 80.01) (xy 252.73 82.55))
+  (wire (pts (xy 252.73 80.01) (xy 252.73 83.82))
     (stroke (width 0) (type default))
   )
@@
     (stroke (width 0) (type default))
   )
-  (wire (pts (xy 238.76 82.55) (xy 242.57 82.55))
-    (stroke (width 0) (type default))
-  )
   (wire (pts (xy 69.85 129.54) (xy 74.93 129.54))
     (stroke (width 0) (type default))
@@
   )
   (wire (pts (xy 69.85 118.11) (xy 74.93 118.11))
-    (stroke (width 0) (type default))
-  )
-  (wire (pts (xy 252.73 82.55) (xy 252.73 83.82))
-    (stroke (width 0) (type default))
-  )
-  (wire (pts (xy 250.19 82.55) (xy 252.73 82.55))
     (stroke (width 0) (type default))
   )
@@
     (property "Intersheetrefs" "${INTERSHEET_REFS}" (at 214.8938 33.02 0)
       (effects (font (size 1.27 1.27)) (justify left) hide)
-    )
-  )
-  (global_label "GND" (shape input) (at 238.76 82.55 180) (fields_autoplaced)
-    (effects (font (size 1.27 1.27)) (justify right))
-    (property "Intersheetrefs" "${INTERSHEET_REFS}" (at 231.9043 82.55 0)
-      (effects (font (size 1.27 1.27)) (justify right) hide)
     )
   )
@@
         )
       )
-    )
-  )
-  (symbol (lib_id "Device:R") (at 246.38 82.55 90) (unit 1)
-    (in_bom yes) (on_board yes) (dnp no) (fields_autoplaced)
-    (property "Reference" "R2" (at 246.38 76.2 90)
-      (effects (font (size 1.27 1.27)))
-    )
-    (property "Value" "100K" (at 246.38 78.74 90)
-      (effects (font (size 1.27 1.27)))
-    )
-    (property "Footprint" "Resistor_SMD:R_1206_3216Metric" (at 246.38 84.328 90)
-      (effects (font (size 1.27 1.27)) hide)
-    )
-    (property "Datasheet" "~" (at 246.38 82.55 0)
-      (effects (font (size 1.27 1.27)) hide)
-    )
-    (pin "1")
-    (pin "2")
-    (instances
-      (project "xiao_lamp"
-        (path "/afe119bb-39d8-41a8-9c9c-1156846e84f7"
-          (reference "R2") (unit 1)
-        )
-      )

Commit message: добавлены файлы на печать
Other:
- company: (none) -> LotauRus
- title: (none) -> XIAO LAMP
Changed lines of the file:
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@@
 (kicad_sch (version 20230121) (generator eeschema)
   (paper "A4")
+  (title_block
+    (title "XIAO LAMP")
+    (date "2023-10-02")
+    (rev "12")
+    (company "LotauRus")
+  )
   (junction (at 248.92 38.1) (diameter 0) (color 0 0 0 0)
   )
